Commit message: minor update

File: project_ws/src/my_robot_description/urdf/robot.urdf (robot description, URDF)
Before this commit: robot Robot1, 12 links, 11 joints
Joints:
- joint base_to_wheel1: type fixed -> continuous
- joint base_to_wheel2: type fixed -> continuous
- joint base_to_wheel3: type fixed -> continuous
- joint base_to_wheel4: type fixed -> continuous
